File: Nixie_Controller/Nixie_Controller.brd (EAGLE design)
At the start: 150 x 100 mm, 69 parts, among them IC1 4028N, T1 MMBTA42, T10 MMBTA42, T11 MMBTA42, T12 MMBTA42, T13 MMBTA42, T14 MMBTA42, T15 MMBTA42, T16 MMBTA42, T17 MMBTA42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

Commit message: fix: Reroute traces
Reroute multiple traces for a cleaner look.
Increase the tracewidth of the USB VBUS Signal.
Add decoupling capacitors to the USB supply.
Parts:
- added C11: 1u, resistor:C0805
- added C12: 100n, resistor:C0805
- moved R20 50.1 mm to (36.2, 81.9), turned to 270 degrees
- moved R24 5.08 mm to (64.1, 78.7)
- moved R15 3.86 mm to (139.7, 84.5)
- moved LDR 2.69 mm to (140.6, 91.2), turned to 270 degrees
- moved R16 2.54 mm to (142.9, 73.0)
- moved R19 2.54 mm to (142.9, 78.1)
- moved R17 2.54 mm to (142.9, 75.6)
- moved R2 1.91 mm to (85.7, 67.9)
- moved R3 1.91 mm to (81.9, 67.9)
- moved R4 1.91 mm to (78.1, 67.9)
- moved R5 1.91 mm to (74.3, 67.9)
- moved R6 1.91 mm to (70.5, 67.9)
- moved R7 1.91 mm to (66.7, 67.9)
- moved T2 1.91 mm to (85.1, 63.5)
- moved T3 1.91 mm to (81.3, 63.5)
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Connections:
- net GND: now also C11.2, C12.2
- net VDD: now also C11.1, C12.1
Routing:
- net 3V3@2: track 93.3 -> 155.7 mm
- net +3V3: track 113.0 -> 51.3 mm
- net N$88: track 32.2 -> 42.0 mm
- net N$103: track 57.0 -> 50.6 mm
- net VDD: track 311.0 -> 306.3 mm
- net N$94: track 82.9 -> 85.4 mm
- net N$2: track 24.9 -> 27.2 mm
- net +170V: track 185.2 -> 182.9 mm
- net N$26: track 130.0 -> 127.9 mm
- net N$22: track 158.4 -> 156.5 mm
- net N$25: track 129.4 -> 127.5 mm
- net N$4: track 25.5 -> 27.4 mm
- net N$6: track 17.9 -> 19.8 mm
- net N$5: track 27.3 -> 29.2 mm
- net N$3: track 27.4 -> 29.3 mm
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
Commit message: feat: Generate Gerberfiles
Routing:
- net +3V3: track 51.3 -> 52.6 mm
- net GND: track 15.0 -> 16.3 mm
- net +24V: track 18.6 -> 19.8 mm
- net +12V: track 25.3 -> 26.6 mm
- net VDD: track 306.3 -> 307.5 mm
Changed lines of the file:
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@@
 <drawing>
 <settings>
-<setting alwaysvectorfont="yes"/>
+<setting alwaysvectorfont="no"/>
 <setting keepoldvectorfont="yes"/>
 <setting verticaltext="up"/>
@@
 <layer number="19" name="Unrouted" color="6" fill="1" visible="yes" active="yes"/>
 <layer number="20" name="Dimension" color="24" fill="1" visible="yes" active="yes"/>
-<layer number="21" name="tPlace" color="7" fill="1" visible="yes" active="yes"/>
-<layer number="22" name="bPlace" color="7" fill="1" visible="yes" active="yes"/>
+<layer number="21" name="tPlace" color="7" fill="1" visible="no" active="yes"/>
+<layer number="22" name="bPlace" color="7" fill="1" visible="no" active="yes"/>
 <layer number="23" name="tOrigins" color="15" fill="1" visible="yes" active="yes"/>
 <layer number="24" name="bOrigins" color="15" fill="1" visible="yes" active="yes"/>
@@
 <wire x1="80.645" y1="95.885" x2="78.486" y2="98.044" width="0.6096" layer="1"/>
 <wire x1="78.486" y1="98.044" x2="60.579" y2="98.044" width="0.6096" layer="1"/>
-<wire x1="13.97" y1="88.9" x2="10.795" y2="88.9" width="0.6096" layer="1"/>
-<via x="10.795" y="88.9" extent="1-16" drill="0.55" diameter="1.3"/>
+<wire x1="13.97" y1="88.9" x2="9.525" y2="88.9" width="0.6096" layer="1"/>
+<via x="9.525" y="88.9" extent="1-16" drill="0.55" diameter="1.3"/>
 <wire x1="141.224" y1="98.171" x2="143.725" y2="95.67" width="0.6096" layer="1"/>
 <wire x1="143.725" y1="95.67" x2="143.725" y2="78.105" width="0.6096" layer="1"/>
@@
 <wire x1="12.694" y1="6.811" x2="12.744" y2="6.861" width="0.2032" layer="1"/>
 <wire x1="12.744" y1="6.861" x2="12.744" y2="8.031" width="0.2032" layer="1"/>
-<wire x1="13.97" y1="83.82" x2="10.795" y2="83.82" width="0.6096" layer="1"/>
-<via x="10.795" y="83.82" extent="1-16" drill="0.55" diameter="1.3"/>
+<wire x1="13.97" y1="83.82" x2="9.525" y2="83.82" width="0.6096" layer="1"/>
+<via x="9.525" y="83.82" extent="1-16" drill="0.55" diameter="1.3"/>
 <contactref element="C12" pad="2"/>
 <contactref element="C11" pad="2"/>
 <contactref element="C1" pad="2"/>
 <contactref element="C10" pad="2"/>
-<wire x1="129.54" y1="80.645" x2="140.589" y2="94.996" width="0" layer="19" extent="1-1"/>
-<wire x1="124.46" y1="95.885" x2="129.54" y2="80.645" width="0" layer="19" extent="1-1"/>
-<wire x1="84.14" y1="64.6" x2="129.54" y2="80.645" width="0" layer="19" extent="1-1"/>
-<wire x1="80.33" y1="64.6" x2="84.14" y2="64.6" width="0" layer="19" extent="1-1"/>
-<wire x1="76.52" y1="64.6" x2="80.33" y2="64.6" width="0" layer="19" extent="1-1"/>
-<wire x1="72.71" y1="64.6" x2="76.52" y2="64.6" width="0" layer="19" extent="1-1"/>
-<wire x1="68.9" y1="64.6" x2="72.71" y2="64.6" width="0" layer="19" extent="1-1"/>
-<wire x1="65.09" y1="64.6" x2="68.9" y2="64.6" width="0" layer="19" extent="1-1"/>
-<wire x1="73.025" y1="78.105" x2="72.71" y2="64.6" width="0" layer="19" extent="1-1"/>
-<wire x1="59.375" y1="79.84" x2="73.025" y2="78.105" width="0" layer="19" extent="1-1"/>
-<wire x1="55.565" y1="79.84" x2="59.375" y2="79.84" width="0" layer="19" extent="1-1"/>
-<wire x1="51.755" y1="79.84" x2="55.565" y2="79.84" width="0" layer="19" extent="1-1"/>
-<wire x1="47.945" y1="79.84" x2="51.755" y2="79.84" width="0" layer="19" extent="1-1"/>
-<wire x1="38.735" y1="95.885" x2="47.945" y2="79.84" width="0" layer="19" extent="1-1"/>
-<wire x1="26.67" y1="90.49" x2="38.735" y2="95.885" width="0" layer="19" extent="1-1"/>
-<wire x1="23.495" y1="90.49" x2="26.67" y2="90.49" width="0" layer="19" extent="1-1"/>
-<wire x1="20.32" y1="89.85" x2="23.495" y2="90.49" width="0" layer="19" extent="1-1"/>
-<wire x1="17.78" y1="89.85" x2="20.32" y2="89.85" width="0" layer="19" extent="1-1"/>
-<wire x1="20.32" y1="83.505" x2="20.32" y2="89.85" width="0" layer="19" extent="1-1"/>
-<wire x1="17.78" y1="83.505" x2="20.32" y2="83.505" width="0" layer="19" extent="1-1"/>
-<wire x1="13.97" y1="83.82" x2="17.78" y2="83.505" width="0" layer="19" extent="1-1"/>
-<wire x1="20.32" y1="96.2" x2="20.32" y2="89.85" width="0" layer="19" extent="1-1"/>
-<wire x1="17.78" y1="96.2" x2="20.32" y2="96.2" width="0" layer="19" extent="1-1"/>
-<wire x1="65.847" y1="33.782" x2="65.09" y2="64.6" width="0" layer="19" extent="1-1"/>
-<wire x1="65.847" y1="31.369" x2="65.847" y2="33.782" width="0" layer="19" extent="1-1"/>
-<wire x1="66.675" y1="27.305" x2="65.847" y2="31.369" width="0" layer="19" extent="1-1"/>
-<wire x1="61.595" y1="27.305" x2="66.675" y2="27.305" width="0" layer="19" extent="1-1"/>
-<wire x1="51.435" y1="31.75" x2="61.595" y2="27.305" width="0" layer="19" extent="1-1"/>
-<wire x1="48.895" y1="31.75" x2="51.435" y2="31.75" width="0" layer="19" extent="1-1"/>
-<wire x1="30.734" y1="23.876" x2="48.895" y2="31.75" width="0" layer="19" extent="1-1"/>
-<wire x1="30.734" y1="21.336" x2="30.734" y2="23.876" width="0" layer="19" extent="1-1"/>
-<wire x1="34.08" y1="8.031" x2="30.734" y2="21.336" width="0" layer="19" extent="1-1"/>
-<wire x1="32.34" y1="1.821" x2="32.7" y2="6.211" width="0" layer="19" extent="1-1"/>
-<wire x1="39.58" y1="8.031" x2="34.08" y2="8.031" width="0" layer="19" extent="1-1"/>
-<wire x1="41.32" y1="1.821" x2="40.845" y2="6.096" width="0" layer="19" extent="1-1"/>
-<wire x1="48.895" y1="3.81" x2="41.32" y2="1.821" width="0" layer="19" extent="1-1"/>
-<wire x1="51.435" y1="3.81" x2="48.895" y2="3.81" width="0" layer="19" extent="1-1"/>
-<wire x1="19.984" y1="1.821" x2="32.34" y2="1.821" width="0" layer="19" extent="1-1"/>
-<wire x1="19.624" y1="6.211" x2="19.984" y2="1.821" width="0" layer="19" extent="1-1"/>
-<wire x1="12.744" y1="8.031" x2="18.244" y2="8.031" width="0" layer="19" extent="1-1"/>
-<wire x1="11.004" y1="1.821" x2="11.364" y2="6.211" width="0" layer="19" extent="1-1"/>
-<wire x1="15.941" y1="34.29" x2="11.004" y2="1.821" width="0" layer="19" extent="1-1"/>
-<wire x1="15.941" y1="31.75" x2="15.941" y2="34.29" width="0" layer="19" extent="1-1"/>
-<wire x1="2.794" y1="21.336" x2="12.744" y2="8.031" width="0" layer="19" extent="1-1"/>
-<wire x1="2.794" y1="23.876" x2="2.794" y2="21.336" width="0" layer="19" extent="1-1"/>
-<wire x1="83.705" y1="5.885" x2="66.675" y2="27.305" width="0" layer="19" extent="1-1"/>
-<wire x1="91.325" y1="3.345" x2="83.705" y2="5.885" width="0" layer="19" extent="1-1"/>
-<wire x1="96.405" y1="3.345" x2="91.325" y2="3.345" width="0" layer="19" extent="1-1"/>
-<wire x1="101.485" y1="5.885" x2="96.405" y2="3.345" width="0" layer="19" extent="1-1"/>
-<wire x1="109.105" y1="3.345" x2="101.485" y2="5.885" width="0" layer="19" extent="1-1"/>
-<wire x1="116.725" y1="3.345" x2="109.105" y2="3.345" width="0" layer="19" extent="1-1"/>
-<wire x1="121.805" y1="5.885" x2="116.725" y2="3.345" width="0" layer="19" extent="1-1"/>
-<wire x1="126.885" y1="5.885" x2="121.805" y2="5.885" width="0" layer="19" extent="1-1"/>
-<wire x1="126.885" y1="3.345" x2="126.885" y2="5.885" width="0" layer="19" extent="1-1"/>
 </signal>
 <signal name="N$21">
@@
 <wire x1="36.195" y1="93.98" x2="37.465" y2="92.71" width="0.6096" layer="1"/>
 <wire x1="37.465" y1="92.71" x2="46.14" y2="92.71" width="0.6096" layer="1"/>
-<wire x1="13.97" y1="86.36" x2="10.795" y2="86.36" width="0.6096" layer="1"/>
-<via x="10.795" y="86.36" extent="1-16" drill="0.55" diameter="1.3"/>
+<wire x1="13.97" y1="86.36" x2="9.525" y2="86.36" width="0.6096" layer="1"/>
+<via x="9.525" y="86.36" extent="1-16" drill="0.55" diameter="1.3"/>
 <wire x1="36.195" y1="85.405" x2="36.195" y2="82.765" width="0.6096" layer="1"/>
 </signal>
@@
 <wire x1="30.8" y1="93.345" x2="31.115" y2="93.345" width="0.3048" layer="1"/>
 <via x="31.115" y="93.345" extent="1-16" drill="0.55" diameter="1.3"/>
-<wire x1="13.97" y1="91.44" x2="10.795" y2="91.44" width="0.6096" layer="1"/>
-<via x="10.795" y="91.44" extent="1-16" drill="0.55" diameter="1.3"/>
+<wire x1="13.97" y1="91.44" x2="9.525" y2="91.44" width="0.6096" layer="1"/>
+<via x="9.525" y="91.44" extent="1-16" drill="0.55" diameter="1.3"/>
 </signal>
 <signal name="N$44">
@@
 <wire x1="22.545" y1="94.3" x2="24.13" y2="95.885" width="0.6096" layer="1"/>
 <via x="24.13" y="95.885" extent="1-16" drill="0.55" diameter="1.3"/>
-<wire x1="13.97" y1="93.98" x2="10.795" y2="93.98" width="0.6096" layer="1"/>
-<via x="10.795" y="93.98" extent="1-16" drill="0.55" diameter="1.3"/>
+<wire x1="13.97" y1="93.98" x2="9.525" y2="93.98" width="0.6096" layer="1"/>
+<via x="9.525" y="93.98" extent="1-16" drill="0.55" diameter="1.3"/>
 </signal>
 <signal name="N$43">
